File: SuperRGB.kicad_pcb (KiCad board)
At the start: 2 copper layers, 56.3 x 248.9 mm, 83 parts, among them J1 Conn_01x15, J2 RJ45-TRANSFO, J3 Barrel_Jack, J4 Conn_01x40, J5 Audio-Jack-4, J6 USB_A, M1 V3S, U1 MIC23450, U2 AP1501, U3 NCP114SN, Y1 24MHz, Y2 32768

Commit message: almost complete schematic, preliminary unrouted layout
Parts:
- removed M1: V3S, Package_QFP:LQFP-128_14x14mm_P0.4mm
- added C28: 1u, Capacitor_SMD:C_0603_1608Metric, F.Cu at (60.2, 100.2)
- added C29: 1u, Capacitor_SMD:C_0603_1608Metric, F.Cu at (72.3, 120.8)
- added C30: 100n, Capacitor_SMD:C_0603_1608Metric, B.Cu at (59.5, 116.2)
- added C31: 100n, Capacitor_SMD:C_0603_1608Metric, B.Cu at (60.1, 110.7)
- added C32: 100n, Capacitor_SMD:C_0603_1608Metric, F.Cu at (59.4, 104.5)
- added C48: 100n, Capacitor_SMD:C_0603_1608Metric, B.Cu at (62.9, 107.8)
- added J7: Micro_SD_Card, Connector_Card:microSD_HC_Wuerth_693072010801, F.Cu at (48.9, 80.7)
- added U4: V3S_QFP-128, Package_QFP:LQFP-128_14x14mm_P0.4mm, F.Cu at (64.5, 113.8)
- added U5: GD5F1GQ4UAYIG, Package_SOIC:SOIC-8-1EP_3.9x4.9mm_P1.27mm, F.Cu at (79.1, 125.2)
- C16, C22, C23, C24, C33, C34, C35, C36, C39, C40, C41, C42, C43, C44: moved to B.Cu
- L1: footprint Inductor_SMD:L_6.3x6.3_H3 -> Inductor_SMD:L_0805_2012Metric
- moved C21 167.3 mm to (79.8, 138.9)
- moved C17 165.6 mm to (82.6, 137.7), turned to 90 degrees
- moved C20 149.3 mm to (86.4, 141.0), turned to 90 degrees
- moved R21 135.8 mm to (40.3, 165.7), turned to 90 degrees
- moved L1 118.0 mm to (43.4, 191.4), turned to 270 degrees
- moved C18 117.5 mm to (51.4, 194.1)
- moved R7 109.2 mm to (52.0, 197.7)
- moved C9 106.7 mm to (74.7, 137.1), turned to 90 degrees
- moved R9 106.5 mm to (51.5, 184.5)
- moved R11 106.2 mm to (62.5, 187.5)
- moved Y2 105.1 mm to (67.4, 100.6), turned to 135 degrees
- moved R10 104.4 mm to (59.0, 185.2), turned to 180 degrees
- moved C13 96.1 mm to (86.8, 191.3), turned to 225 degrees
- moved R6 95.8 mm to (54.2, 188.8)
- moved R8 95.5 mm to (53.9, 181.3)
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Connections:
- C11 pad 1: GNDPWR -> GND
- C13 pad 1: GNDPWR -> GND
- C15 pad 1: GNDPWR -> GND
- C17 pad 2: GNDPWR -> GND
- C20 pad 2: GNDPWR -> GND
- C21 pad 2: GNDPWR -> GND
- C22 pad 2: GNDPWR -> GND
- C23 pad 2: GNDPWR -> GND
- C24 pad 2: GNDPWR -> GND
- C25 pad 2: GNDPWR -> GND
- C26 pad 2: GNDPWR -> GND
- C9 pad 2: GNDA -> GND
- D1 pad 2: GNDPWR -> GND
- J3 pad 1: +12V -> Net-(D2-Pad2)
- J3 pad 2: GNDPWR -> GND
- J3 pad 3: GNDPWR -> GND
- R14 pad 1: /PWR_GOOD -> /RESET
- R16 pad 1: GNDA -> GND
- R17 pad 1: GNDA -> GND
- R18 pad 1: GNDA -> GND
- U1 pad 1: /PWR_GOOD -> /RESET
- U1 pad 11: GNDA -> GND
- U1 pad 12: /PWR_GOOD -> /RESET
- U1 pad 18: GNDPWR -> GND
- U1 pad 2: GNDA -> GND
- U1 pad 22: GNDPWR -> GND
- U1 pad 24: GNDPWR -> GND
- U1 pad 6: /PWR_GOOD -> /RESET
- U1 pad 7: GNDA -> GND
- U2 pad 3: GNDPWR -> GND
- U2 pad 5: GNDPWR -> GND
Routing:
- net /DCLK: track 52.7 -> 0.33 mm
- net /HSYNC: track 45.8 -> 0.00 mm
- net /ENAB: track 45.8 -> 0.00 mm, vias 2 -> 0
- net /VSYNC: track 43.3 -> 0.01 mm
- net /B1: track 38.0 -> 0.00 mm, vias 2 -> 0
- net /R1: track 38.0 -> 0.00 mm, vias 2 -> 0
- net /R2: track 37.4 -> 0.00 mm, vias 2 -> 0
- net /B2: track 37.2 -> 0.00 mm, vias 2 -> 0
- net /R3: track 36.4 -> 0.00 mm, vias 2 -> 0
- net /B5: track 35.6 -> 0.00 mm, vias 2 -> 0
- net /R4: track 35.1 -> 0.00 mm, vias 2 -> 0
- net /R5: track 34.2 -> 0.00 mm, vias 2 -> 0
- net +1V8: track 16.3 -> 2.31 mm, vias 3 -> 1
- net Net-(C9-Pad1): track 0.00 -> 13.9 mm, vias 0 -> 3
- net Net-(C7-Pad1): track 0.00 -> 9.31 mm, vias 0 -> 1
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- removed copper zone on B.Cu, net GND

Commit message: finished schematic for my V3s evaluation board
Parts:
- added C49: 4u7, Capacitor_SMD:C_0805_2012Metric_Pad1.15x1.50mm_HandSolder, F.Cu at (84.9, 53.0)
- added C50: 4u7, Capacitor_SMD:C_0805_2012Metric_Pad1.15x1.50mm_HandSolder, F.Cu at (84.9, 58.7)
- added C51: 1u, Capacitor_SMD:C_0805_2012Metric_Pad1.15x1.50mm_HandSolder, F.Cu at (79.9, 59.8)
- added C52: 4u7, Capacitor_SMD:C_0805_2012Metric_Pad1.15x1.50mm_HandSolder, F.Cu at (75.7, 59.8)
- added C53: 1u, Capacitor_SMD:C_0603_1608Metric, F.Cu at (24.3, 99.7)
- added C54: 1p, Capacitor_SMD:C_0603_1608Metric, F.Cu at (9.76, 101.8)
- added C55: 1p2, Capacitor_SMD:C_0603_1608Metric, F.Cu at (13.2, 101.8)
- added C56: 10p, Capacitor_SMD:C_0603_1608Metric, F.Cu at (16.7, 101.8)
- added C57: 2n7, Capacitor_SMD:C_0603_1608Metric, F.Cu at (9.76, 107.1)
- added D2: SS34, Diode_SMD:D_SMA-SMB_Universal_Handsoldering, F.Cu at (13.2, 95.0)
- added D3: SB120, Diode_SMD:D_SOD-123, F.Cu at (77.1, 48.1)
- added D4: SB120, Diode_SMD:D_SOD-123, F.Cu at (71.0, 58.7)
- added J8: Conn_01x12_Male, Connector_PinHeader_2.54mm:PinHeader_1x12_P2.54mm_Vertical, F.Cu at (112.2, 156.6)
- added J9: Conn_01x10, Connector_FFC-FPC:Hirose_FH12-10S-0.5SH_1x10_P0.50mm_Horizontal, F.Cu at (64.1, 41.2)
- added L6: L_Core_Ferrite, Inductor_SMD:L_Taiyo-Yuden_NR-40xx_HandSoldering, F.Cu at (75.5, 40.5)
- added L7: L_Core_Ferrite, Inductor_SMD:L_Taiyo-Yuden_NR-40xx_HandSoldering, F.Cu at (62.8, 53.2)
- added NT1: Net-Tie_2, NetTie:NetTie-2_SMD_Pad2.0mm, F.Cu at (22.4, 94.0)
- added R22: 0.68, Resistor_SMD:R_0805_2012Metric_Pad1.15x1.50mm_HandSolder, F.Cu at (83.1, 47.2)
- added R23: 1, Resistor_SMD:R_0805_2012Metric_Pad1.15x1.50mm_HandSolder, F.Cu at (89.2, 39.4)
- added R24: 1, Resistor_SMD:R_0805_2012Metric_Pad1.15x1.50mm_HandSolder, F.Cu at (76.5, 54.1)
- added R25: 1, Resistor_SMD:R_0805_2012Metric_Pad1.15x1.50mm_HandSolder, F.Cu at (87.3, 47.2)
- added R28: 6.18, Resistor_SMD:R_0805_2012Metric_Pad1.15x1.50mm_HandSolder, F.Cu at (80.7, 54.1)
- C17, C20, C21: value 4u7 -> 10u
- C22, C23, C24: value 100n -> 220p; moved to F.Cu
- C29: value 1u -> 10u
- C9: value 100n -> 1u
- R13: value 50 -> 100k; footprint Resistor_SMD:R_0603_1608Metric -> Resistor_SMD:R_0603_1608Metric_Pad0.84x1.00mm_HandSolder
- R14: value 10k -> 100k; footprint Resistor_SMD:R_0603_1608Metric -> Resistor_SMD:R_0603_1608Metric_Pad0.84x1.00mm_HandSolder
- R15: value 301k -> 100k
- R16, R17: value 158k -> 100k
- R18: value 158k -> 110k
- R19: value 301k -> 150k
- R20: value 301k -> 510k
- U1: value MIC23450 -> EA3036; footprint Package_DFN_QFN:QFN-32-1EP_5x5mm_P0.5mm -> Package_DFN_QFN:UQFN-20-1EP_3x3mm_P0.4mm
- moved J5 112.9 mm to (44.2, 97.6), turned to 225 degrees
- moved R14 76.3 mm to (20.5, 99.7), turned to 0 degrees
- moved C22 62.6 mm to (113.3, 141.2), turned to 0 degrees
- moved R13 62.3 mm to (28.6, 93.6), turned to 0 degrees
- moved C13 60.4 mm to (108.9, 135.1), turned to 0 degrees
- moved C24 52.3 mm to (114.7, 128.6), turned to 180 degrees
- moved L4 50.1 mm to (118.4, 130.8)
- moved C23 45.0 mm to (111.4, 130.1), turned to 0 degrees
- moved R27 44.9 mm to (82.9, 109.9)
- moved R26 44.9 mm to (84.6, 109.8)
- moved L3 41.6 mm to (107.7, 130.5), turned to 90 degrees
- moved C9 40.9 mm to (115.6, 137.7)
- moved R18 38.8 mm to (114.7, 131.7), turned to 180 degrees
- moved U1 38.5 mm to (112.7, 134.9), turned to 270 degrees
- moved L2 37.9 mm to (109.7, 140.4)
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Connections:
- net /LCD_BL_R renamed RLED_CTRL
- net /LCD_BL_W renamed WLED_CTRL
- C11 pad 2: VBUS -> +5V
- C13 pad 2: VBUS -> +5V
- C15 pad 2: VBUS -> +5V
- C22 pad 2: GND -> Net-(C22-Pad2)
- C23 pad 2: GND -> Net-(C23-Pad2)
- C24 pad 2: GND -> Net-(C24-Pad2)
- C26 pad 1: VBUS -> +5V
- C9 pad 1: Net-(C9-Pad1) -> +5V
- J6 pad 1: VBUS -> +5V
- L5 pad 2: VBUS -> +5V
- R13 pad 1: Net-(C9-Pad1) -> +3V3
- R13 pad 2: VBUS -> Net-(R13-Pad2)
- R14 pad 1: /RESET -> +3V3
- R14 pad 2: +3V3 -> Net-(R13-Pad2)
- R15 pad 2: Net-(R15-Pad2) -> Net-(C22-Pad2)
- R16 pad 2: Net-(R15-Pad2) -> Net-(C22-Pad2)
- R17 pad 2: Net-(R17-Pad2) -> Net-(C23-Pad2)
- R18 pad 2: Net-(R18-Pad2) -> Net-(C24-Pad2)
- R19 pad 2: Net-(R17-Pad2) -> Net-(C23-Pad2)
- R20 pad 2: Net-(R18-Pad2) -> Net-(C24-Pad2)
- U1 pad 1: /RESET -> GND
- U1 pad 10: Net-(R18-Pad2) -> +5V
- U1 pad 11: GND -> Net-(L2-Pad1)
- U1 pad 12: /RESET -> GND
- U1 pad 13: Net-(C9-Pad1) -> GND
- U1 pad 14: VBUS -> Net-(C22-Pad2)
- U1 pad 15: Net-(C9-Pad1) -> GND
- U1 pad 16: (no net) -> +5V
- U1 pad 17: (no net) -> GND
- U1 pad 18: GND -> +5V
- U1 pad 19: (no net) -> +5V
- U1 pad 2: GND -> Net-(C24-Pad2)
- U1 pad 20: (no net) -> Net-(L4-Pad1)
- U1 pad 21: Net-(L4-Pad1) -> GND
- U1 pad 3: VBUS -> Net-(C23-Pad2)
- U1 pad 4: +1V8 -> GND
- U1 pad 5: Net-(R17-Pad2) -> GND
- U1 pad 6: /RESET -> Net-(L3-Pad1)
- U1 pad 7: GND -> +5V
- U1 pad 8: VBUS -> +5V
- U1 pad 9: +1V2 -> +5V
- U2 pad 4: VBUS -> +5V
- U3 pad 1: VBUS -> +5V
- U3 pad 3: VBUS -> +5V
- U4 pad 100: Net-(U4-Pad100) -> /GPIO0
Routing:
- net +5V: track 0.00 -> 24.4 mm
- net Net-(C9-Pad1): track 13.9 -> 0.00 mm, vias 3 -> 0
- net GND: track 13.1 -> 23.3 mm, vias 4 -> 18
- net Net-(C7-Pad1): track 9.31 -> 0.00 mm, vias 1 -> 0
- net VBUS: track 6.01 -> 0.00 mm
- net Net-(C22-Pad2): track 0.00 -> 5.84 mm
- net Net-(C24-Pad2): track 0.00 -> 5.20 mm
- net Net-(C23-Pad2): track 0.00 -> 5.15 mm
- net Net-(L4-Pad1): track 0.00 -> 5.07 mm
- net /SPI_MOSI: track 4.92 -> 0.00 mm
- net /SPI_MISO: track 4.59 -> 0.00 mm
- net Net-(L3-Pad1): track 0.00 -> 4.40 mm
- net /SPI_SCK: track 4.30 -> 0.00 mm
- net /SPI_CS: track 4.08 -> 0.00 mm
- net +1V8: track 2.31 -> 6.09 mm, vias 1 -> 0
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- added copper zone on B.Cu, net GND
